File: daughter/circuits/audio-amplifier.sch (KiCad schematic (older format))
At the start: 22 parts, among them J10 Conn_01x05, J8 AudioJack_3.5TRS, J9 AudioJack_3.5TRS, U14 TDA7851F

Commit message: complete redesign for GM dash, including hvac replacement
Parts:
- removed R34, R35, R36: R_1k, Resistor_SMD:R_0603_1608Metric_Pad1.05x0.95mm_HandSolder, symbol open-automation:R_1k
- added R24, R25, R26: R_1K, Resistor_SMD:R_0603_1608Metric_Pad0.98x0.95mm_HandSolder, symbol Open_Automation:R_1K
- C10: renamed from C21; footprint Capacitor_SMD:C_0603_1608Metric_Pad1.05x0.95mm_HandSolder -> Capacitor_SMD:C_0603_1608Metric_Pad1.08x0.95mm_HandSolder; symbol open-automation:C_1uF -> Open_Automation:C_1uF; LCSC (none) -> C96446; Part Number GCM188R71C105KA64D -> CL10A106MA8NRNC; Website https://www.digikey.com/product-detail/en/murata-electronic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 -> (none)
- C11: renamed from C22; footprint Capacitor_SMD:C_0603_1608Metric_Pad1.05x0.95mm_HandSolder -> Capacitor_SMD:C_0603_1608Metric_Pad1.08x0.95mm_HandSolder; symbol open-automation:C_1uF -> Open_Automation:C_1uF; LCSC (none) -> C96446; Part Number GCM188R71C105KA64D -> CL10A106MA8NRNC; Website https://www.digikey.com/product-detail/en/murata-electronic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 -> (none)
- C12: renamed from C23; footprint Capacitor_SMD:C_0603_1608Metric_Pad1.05x0.95mm_HandSolder -> Capacitor_SMD:C_0603_1608Metric_Pad1.08x0.95mm_HandSolder; symbol open-automation:C_0.1uF -> Open_Automation:C_0.1uF; LCSC (none) -> C14663; Part Number C1608X8R1H104K080AB -> CC0603KRX7R9BB104
- C13: renamed from C24; footprint Capacitor_SMD:C_0603_1608Metric_Pad1.05x0.95mm_HandSolder -> Capacitor_SMD:C_0603_1608Metric_Pad1.08x0.95mm_HandSolder; symbol open-automation:C_0.1uF -> Open_Automation:C_0.1uF; LCSC (none) -> C14663; Part Number C1608X8R1H104K080AB -> CC0603KRX7R9BB104
- C14: renamed from C25; footprint Capacitor_SMD:C_0603_1608Metric_Pad1.05x0.95mm_HandSolder -> Capacitor_SMD:C_0603_1608Metric_Pad1.08x0.95mm_HandSolder; symbol open-automation:C_0.1uF -> Open_Automation:C_0.1uF; LCSC (none) -> C14663; Part Number C1608X8R1H104K080AB -> CC0603KRX7R9BB104
- C15: renamed from C26; footprint Capacitor_SMD:C_0603_1608Metric_Pad1.05x0.95mm_HandSolder -> Capacitor_SMD:C_0603_1608Metric_Pad1.08x0.95mm_HandSolder; symbol open-automation:C_0.1uF -> Open_Automation:C_0.1uF; LCSC (none) -> C14663; Part Number C1608X8R1H104K080AB -> CC0603KRX7R9BB104
- C16: renamed from C27; value C_47uF -> C_10uF; footprint Capacitor_SMD:C_0603_1608Metric_Pad1.05x0.95mm_HandSolder -> Capacitor_SMD:C_0603_1608Metric_Pad1.08x0.95mm_HandSolder; symbol open-automation:C_47uF -> Open_Automation:C_10uF; LCSC (none) -> C96446; Part Number GRM188R60G476ME15D -> CL10A106MA8NRNC
- C17: renamed from C28; symbol open-automation:C_470uF -> Open_Automation:C_470uF; Supplier https://www.digikey.com/product-detail/en/wurth-electronics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 -> (none)
- C18: renamed from C29; footprint Capacitor_SMD:C_0603_1608Metric_Pad1.05x0.95mm_HandSolder -> Capacitor_SMD:C_0603_1608Metric_Pad1.08x0.95mm_HandSolder; symbol open-automation:C_1uF -> Open_Automation:C_1uF; LCSC (none) -> C96446; Part Number GCM188R71C105KA64D -> CL10A106MA8NRNC; Website https://www.digikey.com/product-detail/en/murata-electronic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 -> (none)
- C19: renamed from C30; value C_0.47uF -> C_470nF; footprint Capacitor_SMD:C_0603_1608Metric_Pad1.05x0.95mm_HandSolder -> Capacitor_SMD:C_0603_1608Metric_Pad1.08x0.95mm_HandSolder; symbol open-automation:C_0.470uF -> Open_Automation:C_470nF; LCSC (none) -> C1623; Part Number 885012206075 -> CL10B474KA8NNNC; Website https://www.mouser.com/ProductDetail/Wurth-Electronics/8850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 -> (none)
- C20: renamed from C31; footprint Capacitor_SMD:C_0603_1608Metric_Pad1.05x0.95mm_HandSolder -> Capacitor_SMD:C_0603_1608Metric_Pad1.08x0.95mm_HandSolder; symbol open-automation:C_0.1uF -> Open_Automation:C_0.1uF; LCSC (none) -> C14663; Part Number C1608X8R1H104K080AB -> CC0603KRX7R9BB104
- J10: renamed from J9; footprint open-automation:AudioJack_SJ1-3525N -> Open_Automation:AudioJack_SJ1-3525N; symbol open-automation:AudioJack_3.5TRS -> Open_Automation:AudioJack_3.5TRS
- J8: footprint open-automation:AudioJack_SJ1-3525N -> Open_Automation:AudioJack_SJ1-3525N; symbol open-automation:AudioJack_3.5TRS -> Open_Automation:AudioJack_3.5TRS
- R21: renamed from R31; footprint Resistor_SMD:R_0603_1608Metric_Pad1.05x0.95mm_HandSolder -> Resistor_SMD:R_0603_1608Metric_Pad0.98x0.95mm_HandSolder; symbol open-automation:R_10K -> Open_Automation:R_10K; LCSC (none) -> C25804; Part Number RC0603JR-0710KL -> 0603WAF1002T5E
- R22: renamed from R32; footprint Resistor_SMD:R_0603_1608Metric_Pad1.05x0.95mm_HandSolder -> Resistor_SMD:R_0603_1608Metric_Pad0.98x0.95mm_HandSolder; symbol open-automation:R_47.5k -> Open_Automation:R_47.5k; LCSC (none) -> C23061; Part Number ERJ-3EKF4752V -> 0603WAF4752T5E
- R23: renamed from R33; value R_1k -> R_1K; footprint Resistor_SMD:R_0603_1608Metric_Pad1.05x0.95mm_HandSolder -> Resistor_SMD:R_0603_1608Metric_Pad0.98x0.95mm_HandSolder; symbol open-automation:R_1k -> Open_Automation:R_1K; LCSC (none) -> C21190
- R27: renamed from R37; footprint Resistor_SMD:R_0603_1608Metric_Pad1.05x0.95mm_HandSolder -> Resistor_SMD:R_0603_1608Metric_Pad0.98x0.95mm_HandSolder; symbol open-automation:R_47.5k -> Open_Automation:R_47.5k; LCSC (none) -> C23061; Part Number ERJ-3EKF4752V -> 0603WAF4752T5E
- U8: renamed from U14; footprint open-automation:Flexiwatt25-V -> Open_Automation:Flexiwatt25-V; symbol open-automation:TDA7851F -> Open_Automation:TDA7851F
- renumbered J10 to J9
Connections:
- wire segments 88 -> 90
