File: daughter/circuits/canbus.sch (KiCad schematic (older format))
At the start: 10 parts, among them U3 MCP2551-I_SN

Commit message: complete redesign for GM dash, including hvac replacement
Parts:
- C24: renamed from C1; footprint Capacitor_SMD:C_0603_1608Metric_Pad1.05x0.95mm_HandSolder -> Capacitor_SMD:C_0603_1608Metric_Pad1.08x0.95mm_HandSolder; symbol open-automation:C_0.1uF -> Open_Automation:C_0.1uF; LCSC (none) -> C14663; Part Number C1608X8R1H104K080AB -> CC0603KRX7R9BB104
- C25: renamed from C2; footprint Capacitor_SMD:C_0603_1608Metric_Pad1.05x0.95mm_HandSolder -> Capacitor_SMD:C_0603_1608Metric_Pad1.08x0.95mm_HandSolder; symbol open-automation:C_560pF -> Open_Automation:C_560pF; LCSC (none) -> C84721; Part Number CC0603KPX7R9BB561 -> CL10B561KB8NNNC
- C26: renamed from C3; footprint Capacitor_SMD:C_0603_1608Metric_Pad1.05x0.95mm_HandSolder -> Capacitor_SMD:C_0603_1608Metric_Pad1.08x0.95mm_HandSolder; symbol open-automation:C_560pF -> Open_Automation:C_560pF; LCSC (none) -> C84721; Part Number CC0603KPX7R9BB561 -> CL10B561KB8NNNC
- D13: renamed from D1; symbol open-automation:PESD1CAN-UX -> Open_Automation:PESD1CAN-UX; LCSC (none) -> C152727
- R79: renamed from R8; footprint Resistor_SMD:R_0603_1608Metric_Pad1.05x0.95mm_HandSolder -> Resistor_SMD:R_0603_1608Metric_Pad0.98x0.95mm_HandSolder; symbol open-automation:R_4K7 -> Open_Automation:R_4K7; LCSC (none) -> C23162; Part Number ERJ-3GEYJ472V -> 0603WAF4701T5E
- R80: renamed from R9; footprint Resistor_SMD:R_0603_1608Metric_Pad1.05x0.95mm_HandSolder -> Resistor_SMD:R_0603_1608Metric_Pad0.98x0.95mm_HandSolder; symbol open-automation:R_10K -> Open_Automation:R_10K; LCSC (none) -> C25804; Part Number RC0603JR-0710KL -> 0603WAF1002T5E
- R81: renamed from R1; footprint Resistor_SMD:R_0603_1608Metric_Pad1.05x0.95mm_HandSolder -> Resistor_SMD:R_0603_1608Metric_Pad0.98x0.95mm_HandSolder; symbol open-automation:R_4K7 -> Open_Automation:R_4K7; LCSC (none) -> C23162; Part Number ERJ-3GEYJ472V -> 0603WAF4701T5E
- R82: renamed from R2; footprint Resistor_SMD:R_0603_1608Metric_Pad1.05x0.95mm_HandSolder -> Resistor_SMD:R_0603_1608Metric_Pad0.98x0.95mm_HandSolder; symbol open-automation:R_100 -> Open_Automation:R_100; LCSC (none) -> C84721; Part Number RC0603JR-07100RL -> CL10B561KB8NNNC
- R83: renamed from R3; footprint Resistor_SMD:R_0603_1608Metric_Pad1.05x0.95mm_HandSolder -> Resistor_SMD:R_0603_1608Metric_Pad0.98x0.95mm_HandSolder; symbol open-automation:R_100 -> Open_Automation:R_100; LCSC (none) -> C84721; Part Number RC0603JR-07100RL -> CL10B561KB8NNNC
- U15: renamed from U3; LCSC (none) -> C7376
