File: daughter/circuits/microcontroller.sch (KiCad schematic (older format))
At the start: 18 parts, among them J7 Conn_02x05_Odd_Even, SW1 SW_PUSH, SW2 SW_PUSH, SW3 SW_PUSH, U12 ESP-WROOM-32, U13 SI7020-A20

Commit message: complete redesign for GM dash, including hvac replacement
Parts:
- removed J7: Conn_02x05_Odd_Even, Connector_PinHeader_2.54mm:PinHeader_2x05_P2.54mm_Vertical, symbol open-automation:Conn_02x05_Odd_Even
- removed U12: ESP-WROOM-32, open-automation:ESP-WROOM-32, symbol open-automation:ESP-WROOM-32
- removed U13: SI7020-A20, open-automation:SI7020-A20, symbol open-automation:SI7020-A20
- added U13: ESP32-WROOM-32, RF_Module:ESP32-WROOM-32, symbol Open_Automation:ESP32-WROOM-32
- added U14: Si7020-A20, Package_DFN_QFN:DFN-6-1EP_3x3mm_P1mm_EP1.5x2.4mm, symbol Sensor_Humidity:Si7020-A20
- C21: renamed from C18; footprint Capacitor_SMD:C_0603_1608Metric_Pad1.05x0.95mm_HandSolder -> Capacitor_SMD:C_0603_1608Metric_Pad1.08x0.95mm_HandSolder; symbol open-automation:C_10uF -> Open_Automation:C_10uF; LCSC (none) -> C96446; Part Number GRM188R61E106KA73D -> CL10A106MA8NRNC; Website https://www.mouser.com/ProductDetail/Murata-Electronics/GRM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 -> (none)
- C22: renamed from C19; footprint Capacitor_SMD:C_0603_1608Metric_Pad1.05x0.95mm_HandSolder -> Capacitor_SMD:C_0603_1608Metric_Pad1.08x0.95mm_HandSolder; symbol open-automation:C_1uF -> Open_Automation:C_1uF; LCSC (none) -> C96446; Part Number GCM188R71C105KA64D -> CL10A106MA8NRNC; Website https://www.digikey.com/product-detail/en/murata-electronic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 -> (none)
- C23: renamed from C20; footprint Capacitor_SMD:C_0603_1608Metric_Pad1.05x0.95mm_HandSolder -> Capacitor_SMD:C_0603_1608Metric_Pad1.08x0.95mm_HandSolder; symbol open-automation:C_0.1uF -> Open_Automation:C_0.1uF; LCSC (none) -> C14663; Part Number C1608X8R1H104K080AB -> CC0603KRX7R9BB104
- D10: renamed from D9; symbol open-automation:LED_G -> Open_Automation:LED_G; LCSC (none) -> C72041; Part Number 150060VS75000 -> 19-217/BHC-ZL1M2RY/3T; Website https://www.digikey.com/product-detail/en/wurth-electronics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 -> (none)
- D11: renamed from D10; symbol open-automation:LED_G -> Open_Automation:LED_G; LCSC (none) -> C72041; Part Number 150060VS75000 -> 19-217/BHC-ZL1M2RY/3T; Website https://www.digikey.com/product-detail/en/wurth-electronics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 -> (none)
- D12: renamed from D11; symbol open-automation:LED_G -> Open_Automation:LED_G; LCSC (none) -> C72041; Part Number 150060VS75000 -> 19-217/BHC-ZL1M2RY/3T; Website https://www.digikey.com/product-detail/en/wurth-electronics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 -> (none)
- EN1: renamed from SW1; footprint Button_Switch_SMD:SW_Push_1P1T_NO_CK_KMR2 -> Button_Switch_SMD:SW_SPST_PTS645; symbol open-automation:SW_PUSH -> Open_Automation:SW_PUSH; LCSC (none) -> C127509; Part Number KMR211NG LFS -> K2-1102SP-C4SC-04; Website https://www.digikey.com/product-detail/en/c-k/KMR211NG-LFS/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 -> (none)
- FACT1: renamed from SW3; footprint Button_Switch_SMD:SW_Push_1P1T_NO_CK_KMR2 -> Button_Switch_SMD:SW_SPST_PTS645; symbol open-automation:SW_PUSH -> Open_Automation:SW_PUSH; LCSC (none) -> C127509; Part Number KMR211NG LFS -> K2-1102SP-C4SC-04; Website https://www.digikey.com/product-detail/en/c-k/KMR211NG-LFS/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 -> (none)
- PROG1: renamed from SW2; footprint Button_Switch_SMD:SW_Push_1P1T_NO_CK_KMR2 -> Button_Switch_SMD:SW_SPST_PTS645; symbol open-automation:SW_PUSH -> Open_Automation:SW_PUSH; LCSC (none) -> C127509; Part Number KMR211NG LFS -> K2-1102SP-C4SC-04; Website https://www.digikey.com/product-detail/en/c-k/KMR211NG-LFS/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 -> (none)
- R73: renamed from R25; footprint Resistor_SMD:R_0603_1608Metric_Pad1.05x0.95mm_HandSolder -> Resistor_SMD:R_0603_1608Metric_Pad0.98x0.95mm_HandSolder; symbol open-automation:R_10K -> Open_Automation:R_10K; LCSC (none) -> C25804; Part Number RC0603JR-0710KL -> 0603WAF1002T5E
- R74: renamed from R26; footprint Resistor_SMD:R_0603_1608Metric_Pad1.05x0.95mm_HandSolder -> Resistor_SMD:R_0603_1608Metric_Pad0.98x0.95mm_HandSolder; symbol open-automation:R_10K -> Open_Automation:R_10K; LCSC (none) -> C25804; Part Number RC0603JR-0710KL -> 0603WAF1002T5E
- R75: renamed from R27; footprint Resistor_SMD:R_0603_1608Metric_Pad1.05x0.95mm_HandSolder -> Resistor_SMD:R_0603_1608Metric_Pad0.98x0.95mm_HandSolder; symbol open-automation:R_10K -> Open_Automation:R_10K; LCSC (none) -> C25804; Part Number RC0603JR-0710KL -> 0603WAF1002T5E
- R76: renamed from R28; footprint Resistor_SMD:R_0603_1608Metric_Pad1.05x0.95mm_HandSolder -> Resistor_SMD:R_0603_1608Metric_Pad0.98x0.95mm_HandSolder; symbol open-automation:R_10K -> Open_Automation:R_10K; LCSC (none) -> C25804; Part Number RC0603JR-0710KL -> 0603WAF1002T5E
- R77: renamed from R29; footprint Resistor_SMD:R_0603_1608Metric_Pad1.05x0.95mm_HandSolder -> Resistor_SMD:R_0603_1608Metric_Pad0.98x0.95mm_HandSolder; symbol open-automation:R_10K -> Open_Automation:R_10K; LCSC (none) -> C25804; Part Number RC0603JR-0710KL -> 0603WAF1002T5E
- R78: renamed from R30; footprint Resistor_SMD:R_0603_1608Metric_Pad1.05x0.95mm_HandSolder -> Resistor_SMD:R_0603_1608Metric_Pad0.98x0.95mm_HandSolder; symbol open-automation:R_10K -> Open_Automation:R_10K; LCSC (none) -> C25804; Part Number RC0603JR-0710KL -> 0603WAF1002T5E
Connections:
- net labels added: IO13, IO15, IO16, IO17, IO18, IO19, IO2, IO23, IO25, IO26, IO27, IO32, IO33, IO34, IO35, IO4, IO5
- net labels removed: AUDIO_MUTE, AUDIO_STBY, BATT_IO, CAN_RX, CAN_TX, CURRENT_SENSE, DISPLAY, DISPLAY_EN, MAIN, MAIN_EN, MUTE, Microcontroller, SOFT_POWER, STBY, Temp-Humidty
- wire segments 74 -> 82
