File: daughter/circuits/hvac.sch (KiCad schematic (older format))
At the start: 60 parts, among them Q1 Q_MBT3904, Q10 BC846, Q11 BSS84, Q12 BSS84, Q13 Q_MBT3904, Q14 Q_MBT3904, Q15 Q_DMT3020, Q16 Q_DMT3020, Q2 Q_MBT3904, Q3 Q_DMT3020, Q4 Q_DMT3020, Q5 Q_MBT3904, Q6 Q_MBT3904, Q7 Q_DMT3020, Q8 Q_DMT3020, Q9 BC846, U10 MAX11617, U11 LTV-827S, U9 MCP23017_SS

Commit message: finished layout and routing
Changed lines of the file:
@@
 AIN4
 $Comp
-L open-automation:GND #PWR?
+L open-dash-daughterboard-rescue:GND-open-automation #PWR?
 U 1 1 5FC16751
 P 5550 3100
@@
 	11550 7450 11600 7450
 $Comp
-L open-automation:GND #PWR?
+L open-dash-daughterboard-rescue:GND-open-automation #PWR?
 U 1 1 5FF05705
 P 12350 7700
@@
 	11550 6450 11600 6450
 $Comp
-L open-automation:GND #PWR?
+L open-dash-daughterboard-rescue:GND-open-automation #PWR?
 U 1 1 5FF0572B
 P 12350 6700
@@
 	14600 2200 14550 2200
 $Comp
-L open-automation:GND #PWR?
+L open-dash-daughterboard-rescue:GND-open-automation #PWR?
 U 1 1 5FDA34F9
 P 14600 2500
@@
 	14600 2500 14550 2500
 $Comp
-L open-automation:GND #PWR?
+L open-dash-daughterboard-rescue:GND-open-automation #PWR?
 U 1 1 5FDB34AF
 P 14600 2900
@@
 	14600 2600 14550 2600
 $Comp
-L open-automation:GND #PWR?
+L open-dash-daughterboard-rescue:GND-open-automation #PWR?
 U 1 1 5FE28040
 P 13800 2550
@@
 	13800 2550 13750 2550
 $Comp
-L open-automation:GND #PWR?
+L open-dash-daughterboard-rescue:GND-open-automation #PWR?
 U 1 1 5FE37015
 P 13800 2900
@@
 	14600 3700 14550 3700
 $Comp
-L open-automation:GND #PWR?
+L open-dash-daughterboard-rescue:GND-open-automation #PWR?
 U 1 1 5FFC1633
 P 14600 4000
@@
 	14600 4000 14550 4000
 $Comp
-L open-automation:GND #PWR?
+L open-dash-daughterboard-rescue:GND-open-automation #PWR?
 U 1 1 5FFC163E
 P 14600 4400
@@
 	14600 4100 14550 4100
 $Comp
-L open-automation:GND #PWR?
+L open-dash-daughterboard-rescue:GND-open-automation #PWR?
 U 1 1 5FFC164B
 P 13800 4050
@@
 	13800 4050 13750 4050
 $Comp
-L open-automation:GND #PWR?
+L open-dash-daughterboard-rescue:GND-open-automation #PWR?
 U 1 1 5FFC1656
 P 13800 4400
@@
 	9100 2200 9050 2200
 $Comp
-L open-automation:GND #PWR?
+L open-dash-daughterboard-rescue:GND-open-automation #PWR?
 U 1 1 60044DD0
 P 9100 2500
@@
 	9100 2500 9050 2500
 $Comp
-L open-automation:GND #PWR?
+L open-dash-daughterboard-rescue:GND-open-automation #PWR?
 U 1 1 60044DDB
 P 9100 2900
@@
 	9100 2600 9050 2600
 $Comp
-L open-automation:GND #PWR?
+L open-dash-daughterboard-rescue:GND-open-automation #PWR?
 U 1 1 60044DE8
 P 8300 2550
@@
 	8300 2550 8250 2550
 $Comp
-L open-automation:GND #PWR?
+L open-dash-daughterboard-rescue:GND-open-automation #PWR?
 U 1 1 60044DF3
 P 8300 2900
@@
 	9100 3700 9050 3700
 $Comp
-L open-automation:GND #PWR?
+L open-dash-daughterboard-rescue:GND-open-automation #PWR?
 U 1 1 60044E57
 P 9100 4000
@@
 	9100 4000 9050 4000
 $Comp
-L open-automation:GND #PWR?
+L open-dash-daughterboard-rescue:GND-open-automation #PWR?
 U 1 1 60044E62
 P 9100 4400
@@
 	9100 4100 9050 4100
 $Comp
-L open-automation:GND #PWR?
+L open-dash-daughterboard-rescue:GND-open-automation #PWR?
 U 1 1 60044E6F
 P 8300 4050
@@
 	8300 4050 8250 4050
 $Comp
-L open-automation:GND #PWR?
+L open-dash-daughterboard-rescue:GND-open-automation #PWR?
 U 1 1 60044E7A
 P 8300 4400
@@
 	11800 2200 11750 2200
 $Comp
-L open-automation:GND #PWR?
+L open-dash-daughterboard-rescue:GND-open-automation #PWR?
 U 1 1 600C2937
 P 11800 2500
@@
 	11800 2500 11750 2500
 $Comp
-L open-automation:GND #PWR?
+L open-dash-daughterboard-rescue:GND-open-automation #PWR?
 U 1 1 600C2942
 P 11800 2900
@@
 	11800 2600 11750 2600
 $Comp
-L open-automation:GND #PWR?
+L open-dash-daughterboard-rescue:GND-open-automation #PWR?
 U 1 1 600C294F
 P 11000 2550
@@
 	11000 2550 10950 2550
 $Comp
-L open-automation:GND #PWR?
+L open-dash-daughterboard-rescue:GND-open-automation #PWR?
 U 1 1 600C295A
 P 11000 2900
@@
 	11800 3700 11750 3700
 $Comp
-L open-automation:GND #PWR?
+L open-dash-daughterboard-rescue:GND-open-automation #PWR?
 U 1 1 600C29BE
 P 11800 4000
@@
 	11800 4000 11750 4000
 $Comp
-L open-automation:GND #PWR?
+L open-dash-daughterboard-rescue:GND-open-automation #PWR?
 U 1 1 600C29C9
 P 11800 4400
@@
 	11800 4100 11750 4100
 $Comp
-L open-automation:GND #PWR?
+L open-dash-daughterboard-rescue:GND-open-automation #PWR?
 U 1 1 600C29D6
 P 11000 4050
@@
 	11000 4050 10950 4050
 $Comp
-L open-automation:GND #PWR?
+L open-dash-daughterboard-rescue:GND-open-automation #PWR?
 U 1 1 600C29E1
 P 11000 4400
@@
 $EndComp
 $Comp
-L open-automation:GND #PWR?
+L open-dash-daughterboard-rescue:GND-open-automation #PWR?
 U 1 1 5FD33BAF
 P 9450 6700
@@
 $EndComp
 $Comp
-L open-automation:GND #PWR?
+L open-dash-daughterboard-rescue:GND-open-automation #PWR?
 U 1 1 5FD4BF2F
 P 9450 7100
@@
 	9500 6500 9450 6500
 $Comp
-L open-automation:GND #PWR?
+L open-dash-daughterboard-rescue:GND-open-automation #PWR?
 U 1 1 5FDA2CBB
 P 10150 7100
@@
 	9450 7100 9450 7050
 $Comp
-L open-automation:GND #PWR?
+L open-dash-daughterboard-rescue:GND-open-automation #PWR?
 U 1 1 5FDD129E
 P 10150 6700
@@
 AIN9
 $Comp
-L open-automation:GND #PWR?
+L open-dash-daughterboard-rescue:GND-open-automation #PWR?
 U 1 1 608E2588
 P 5450 7350
