File: daughter/circuits/j1850.sch (KiCad schematic (older format))
At the start: 7 parts, among them U12 LTV-827S

Commit message: finished layout and routing
Changed lines of the file:
@@
 $EndComp
 $Comp
-L open-automation:GND #PWR?
+L open-dash-daughterboard-rescue:GND-open-automation #PWR?
 U 1 1 5FD18EF7
 P 5700 2650
@@
 $EndComp
 $Comp
-L open-automation:GND #PWR?
+L open-dash-daughterboard-rescue:GND-open-automation #PWR?
 U 1 1 5FD18EFD
 P 5700 3050
@@
 	5700 3050 5700 3000
 $Comp
-L open-automation:GND #PWR?
+L open-dash-daughterboard-rescue:GND-open-automation #PWR?
 U 1 1 5FD18F10
 P 6400 2650
