File: daughter/circuits/open-dash-daughterboard.sch (KiCad schematic (older format))
At the start: 6 parts, among them J1 RCA-PJRAN1X1U04X, P1 CONN_01X04, U1 TE-AUTO-CONN-52, U2 radio-housing-mounts

Commit message: complete redesign for GM dash, including hvac replacement
Parts:
- removed J1: RCA-PJRAN1X1U04X, open-automation:RCA-PJRAN1X1U04X, symbol open-automation:RCA-PJRAN1X1U04X
- removed P1: CONN_01X04, Connector_PinHeader_2.54mm:PinHeader_1x04_P2.54mm_Vertical, symbol open-automation:CONN_01X04
- removed R14: R_100K, Resistor_SMD:R_0603_1608Metric_Pad1.05x0.95mm_HandSolder, symbol open-automation:R_100K
- removed R38: R_10K, Resistor_SMD:R_0603_1608Metric_Pad1.05x0.95mm_HandSolder, symbol open-automation:R_10K
- removed U1: TE-AUTO-CONN-52, open-automation:TE-AUTO-CONN-52, symbol open-automation:TE-AUTO-CONN-52
- added D1: D_1N5819HW, Diode_SMD:D_SOD-123, symbol Open_Automation:D_1N5819HW
- added J1: Conn_02x09_Odd_Even, Connector_PinHeader_2.54mm:PinHeader_2x09_P2.54mm_Vertical_SMD, symbol Connector_Generic:Conn_02x09_Odd_Even
- added J2, J3, J4: Molex_Mini-Fit_Jr_5566, Connector_Molex:Molex_Mini-Fit_Jr_5566-24A2_2x12_P4.20mm_Vertical, symbol Open_Automation:Molex_Mini-Fit_Jr_5566
- U1: renamed from U2; footprint open-automation:radio-housing-mounts -> Open_Automation:radio-housing-mounts; symbol open-automation:radio-housing-mounts -> Open_Automation:radio-housing-mounts
Connections:
- net labels added: AIN10, AIN9, AMBIENT_AIR_TEMP, AMBIENT_LIGHT, BATTERY_VOLTAGE_SENSE, BLOWER_MOTOR, DISPLAY_POWER, DRIVER_HEATED_SEAT_STATUS, DRIVER_SEAT_TEMP_CONTROL, DRIVER_SUNLOAD, FACT, IGNITION, IGNITION_SENSE, INSIDE_AIR_TEMP, INSIDE_AIR_TEMP_BLOWER, INSTRUMENT_SUPPLY_VOLTAGE_4, IO13, IO25, IO26, IO27, IO32, J1850, J1850_RX, J1850_TX, LEFT_AIR_TEMP_CONTROL_A, LEFT_AIR_TEMP_CONTROL_B, LOWER_LEFT_AIR_TEMP, LOWER_RIGHT_AIR_TEMP, LOW_REF, MAIN_POWER, MODE_A, MODE_B, OUT11, PASSENGER_HEATED_SEAT_STATUS, PASSENGER_SEAT_TEMP_CONTROL, PASSENGER_SUNLOAD, REAR_DEFOG, RECIRCULATION_A, RECIRCULATION_B, RIGHT_AIR_TEMP_CONTROL_A, RIGHT_AIR_TEMP_CONTROL_B, SENSE1, TRIGGER1, UPPER_LEFT_AIR_TEMP, UPPER_RIGHT_AIR_TEMP, WHEEL_CONTROLS_SIGNAL, WHEEL_CONTROLS_SUPPLY
- net labels removed: BATT_IO, CAMERA+, CAMERA-
- wire segments 73 -> 188
