File: daughter/circuits/power.sch (KiCad schematic (older format))
At the start: 37 parts, among them J11 Barrel_Jack_OD5.5_ID2.5, J5 Barrel_Jack_OD5.5_ID2.5, J6 Barrel_Jack_OD5.5_ID2.5, U10 MIC29302WU, U11 MIC29302WU, U7 ACS711, U8 REG-3.3v, U9 MIC29302WU

Commit message: complete redesign for GM dash, including hvac replacement
Parts:
- removed C10, C12, C13, C14: C_10uF, Capacitor_SMD:C_0603_1608Metric_Pad1.05x0.95mm_HandSolder, symbol open-automation:C_10uF
- removed D3, D4, D5, D6: LED-0603-G, LED_SMD:LED_0603_1608Metric_Pad1.05x0.95mm_HandSolder, symbol open-automation:LED-0603-G
- removed J5, J6: Barrel_Jack_OD5.5_ID2.5, open-automation:BarrelJack_OD5.5_ID2.5, symbol open-automation:Barrel_Jack_OD5.5_ID2.5
- removed R10, R11, R12, R13, R15: R_2.2k, Resistor_SMD:R_0603_1608Metric_Pad1.05x0.95mm_HandSolder, symbol open-automation:R_2.2k
- removed R16, R17, R18: R_20K, Resistor_SMD:R_0603_1608Metric_Pad1.05x0.95mm_HandSolder, symbol open-automation:R_20K
- removed U7: ACS711, Package_SO:SOIC-8_3.9x4.9mm_P1.27mm, symbol open-automation:ACS711
- added C2, C4, C5, C6: C_10uF, Capacitor_SMD:C_0603_1608Metric_Pad1.08x0.95mm_HandSolder, symbol Open_Automation:C_10uF
- added D3, D4, D5, D7: LED_G, LED_SMD:LED_0603_1608Metric_Pad1.05x0.95mm_HandSolder, symbol Open_Automation:LED_G
- added J6, J7: Barrel_Jack_OD5.5_ID2.5, Open_Automation:BarrelJack_OD5.5_ID2.5, symbol Open_Automation:Barrel_Jack_OD5.5_ID2.5
- added R1, R12, R13, R2, R4, R5, R6, R9: R_10K, Resistor_SMD:R_0603_1608Metric_Pad0.98x0.95mm_HandSolder, symbol Open_Automation:R_10K
- added R10, R11, R20, R7, R8: R_1K, Resistor_SMD:R_0603_1608Metric_Pad0.98x0.95mm_HandSolder, symbol Open_Automation:R_1K
- added R3: R_100K, Resistor_SMD:R_0603_1608Metric_Pad0.98x0.95mm_HandSolder, symbol Open_Automation:R_100K
- added U2: LTV-827S, Package_DIP:SMDIP-8_W9.53mm, symbol Open_Automation:LTV-827S
- added U3: ACS711, Sensor_Current:Allegro_QFN-12-10-1EP_3x3mm_P0.5mm, symbol Open_Automation:ACS711
- C1: renamed from C9; symbol open-automation:C_1000uF -> Open_Automation:C_1000uF; Supplier https://www.digikey.com/product-detail/en/panasonic-electro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 -> (none); Website https://www.digikey.com/product-detail/en/panasonic-electro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 -> (none)
- C3: renamed from C11; footprint Capacitor_SMD:C_0603_1608Metric_Pad1.05x0.95mm_HandSolder -> Capacitor_SMD:C_0603_1608Metric_Pad1.08x0.95mm_HandSolder; symbol open-automation:C_10uF -> Open_Automation:C_10uF; LCSC (none) -> C96446; Part Number GRM188R61E106KA73D -> CL10A106MA8NRNC; Website https://www.mouser.com/ProductDetail/Murata-Electronics/GRM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 -> (none)
- C7: renamed from C16; symbol open-automation:C_10uF_Ta -> Open_Automation:C_10uF_Ta; LCSC (none) -> C116748; Part Number TRJC106K035R0600 -> T491C106K025AT
- C8: renamed from C15; symbol open-automation:C_10uF_Ta -> Open_Automation:C_10uF_Ta; LCSC (none) -> C116748; Part Number TRJC106K035R0600 -> T491C106K025AT
- C9: renamed from C17; symbol open-automation:C_10uF_Ta -> Open_Automation:C_10uF_Ta; LCSC (none) -> C116748; Part Number TRJC106K035R0600 -> T491C106K025AT
- D2: symbol open-automation:D_Zener -> Open_Automation:D_Zener; LCSC (none) -> C8835; Part Number SMBJ26CA-H -> SMBJ26CA; Website https://www.mouser.com/ProductDetail/Bourns/SMBJ26CA-H?qs=s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 -> (none)
- D6: renamed from D8; value LED-0603-G -> LED_G; symbol open-automation:LED-0603-G -> Open_Automation:LED_G; LCSC (none) -> C72041; Part Number SML-D12M8WT86 -> 19-217/BHC-ZL1M2RY/3T
- J5: renamed from J11; footprint open-automation:BarrelJack_OD5.5_ID2.5 -> Open_Automation:BarrelJack_OD5.5_ID2.5; symbol open-automation:Barrel_Jack_OD5.5_ID2.5 -> Open_Automation:Barrel_Jack_OD5.5_ID2.5
- R14: renamed from R21; footprint Resistor_SMD:R_0603_1608Metric_Pad1.05x0.95mm_HandSolder -> Resistor_SMD:R_0603_1608Metric_Pad0.98x0.95mm_HandSolder; symbol open-automation:R_20K -> Open_Automation:R_20K; LCSC (none) -> C4184; Part Number RC0603JR-0720KL -> 0603WAF2002T5E
- R15: renamed from R22; value R_6.5k -> R_6.5K; footprint Resistor_SMD:R_0603_1608Metric_Pad1.05x0.95mm_HandSolder -> Resistor_SMD:R_0603_1608Metric_Pad0.98x0.95mm_HandSolder; symbol open-automation:R_6.5k -> Open_Automation:R_6.5K; LCSC (none) -> C23029; Part Number CRCW06036K49FKEAC -> 0603WAF3652T5E; Website https://www.mouser.com/ProductDetail/Vishay-Dale/CRCW06036K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 -> (none)
- R16: renamed from R19; footprint Resistor_SMD:R_0603_1608Metric_Pad1.05x0.95mm_HandSolder -> Resistor_SMD:R_0603_1608Metric_Pad0.98x0.95mm_HandSolder; symbol open-automation:R_20K -> Open_Automation:R_20K; LCSC (none) -> C4184; Part Number RC0603JR-0720KL -> 0603WAF2002T5E
- R17: renamed from R20; value R_2.2k -> R_2.2K; footprint Resistor_SMD:R_0603_1608Metric_Pad1.05x0.95mm_HandSolder -> Resistor_SMD:R_0603_1608Metric_Pad0.98x0.95mm_HandSolder; symbol open-automation:R_2.2k -> Open_Automation:R_2.2K; LCSC (none) -> C4190; Part Number ERJ-3GEYJ222V -> 0603WAF2201T5E
- R18: renamed from R23; footprint Resistor_SMD:R_0603_1608Metric_Pad1.05x0.95mm_HandSolder -> Resistor_SMD:R_0603_1608Metric_Pad0.98x0.95mm_HandSolder; symbol open-automation:R_20K -> Open_Automation:R_20K; LCSC (none) -> C4184; Part Number RC0603JR-0720KL -> 0603WAF2002T5E
- R19: renamed from R24; value R_2.2k -> R_2.2K; footprint Resistor_SMD:R_0603_1608Metric_Pad1.05x0.95mm_HandSolder -> Resistor_SMD:R_0603_1608Metric_Pad0.98x0.95mm_HandSolder; symbol open-automation:R_2.2k -> Open_Automation:R_2.2K; LCSC (none) -> C4190; Part Number ERJ-3GEYJ222V -> 0603WAF2201T5E
- U4: renamed from U8; value REG-3.3v -> REG_3V3; symbol open-automation:REG-3.3v -> Open_Automation:REG_3V3; LCSC (none) -> C152529
- U5: renamed from U10; symbol open-automation:MIC29302WU -> Open_Automation:MIC29302WU; LCSC (none) -> C11149; Part Number MIC29302WU -> MIC29302WU-TR
- U6: renamed from U9; symbol open-automation:MIC29302WU -> Open_Automation:MIC29302WU; LCSC (none) -> C11149; Part Number MIC29302WU -> MIC29302WU-TR
- U7: renamed from U11; symbol open-automation:MIC29302WU -> Open_Automation:MIC29302WU; LCSC (none) -> C11149; Part Number MIC29302WU -> MIC29302WU-TR
Connections:
- net labels added: BATT_ADC, SENSE0, SENSE1, TRIGGER0, TRIGGER1
- wire segments 116 -> 150
Other:
- note removed: "power enable pullups"
