File: daughter/circuits/usb.sch (KiCad schematic (older format))
At the start: 14 parts, among them J4 USB_MINI_B, Q1 Q_NPN_BCE, Q2 Q_PNP_BCE, U6 FT231XS

Commit message: complete redesign for GM dash, including hvac replacement
Parts:
- removed Q1: Q_NPN_BCE, Package_TO_SOT_SMD:SOT-23, symbol Device:Q_NPN_BCE
- removed Q2: Q_PNP_BCE, Package_TO_SOT_SMD:SOT-23, symbol Device:Q_PNP_BEC
- added J12: Conn_02x02_Counter_Clockwise, Connector_PinHeader_2.54mm:PinHeader_2x02_P2.54mm_Vertical, symbol Connector_Generic:Conn_02x02_Counter_Clockwise
- added Q17: Q_NPN, Package_TO_SOT_SMD:SOT-23, symbol Open_Automation:Q_NPN
- added Q18: Q_PNP, Package_TO_SOT_SMD:SOT-23, symbol Open_Automation:Q_PNP
- C27: renamed from C4; footprint Capacitor_SMD:C_0603_1608Metric_Pad1.05x0.95mm_HandSolder -> Capacitor_SMD:C_0603_1608Metric_Pad1.08x0.95mm_HandSolder; symbol open-automation:C_47pF -> Open_Automation:C_47pF; LCSC (none) -> C1671; Part Number GCM1885C2A470FA16D -> CL10C470JB8NNNC
- C28: renamed from C5; footprint Capacitor_SMD:C_0603_1608Metric_Pad1.05x0.95mm_HandSolder -> Capacitor_SMD:C_0603_1608Metric_Pad1.08x0.95mm_HandSolder; symbol open-automation:C_47pF -> Open_Automation:C_47pF; LCSC (none) -> C1671; Part Number GCM1885C2A470FA16D -> CL10C470JB8NNNC
- C29: renamed from C6; footprint Capacitor_SMD:C_0603_1608Metric_Pad1.05x0.95mm_HandSolder -> Capacitor_SMD:C_0603_1608Metric_Pad1.08x0.95mm_HandSolder; symbol open-automation:C_0.1uF -> Open_Automation:C_0.1uF; LCSC (none) -> C14663; Part Number C1608X8R1H104K080AB -> CC0603KRX7R9BB104
- C30: renamed from C7; footprint Capacitor_SMD:C_0603_1608Metric_Pad1.05x0.95mm_HandSolder -> Capacitor_SMD:C_0603_1608Metric_Pad1.08x0.95mm_HandSolder; symbol open-automation:C_4.7uF -> Open_Automation:C_4.7uF; LCSC (none) -> C69335; Part Number C1608X7S0J475K080AC -> CL10A475KA8NQNC
- C31: renamed from C8; footprint Capacitor_SMD:C_0603_1608Metric_Pad1.05x0.95mm_HandSolder -> Capacitor_SMD:C_0603_1608Metric_Pad1.08x0.95mm_HandSolder; symbol open-automation:C_0.1uF -> Open_Automation:C_0.1uF; LCSC (none) -> C14663; Part Number C1608X8R1H104K080AB -> CC0603KRX7R9BB104
- D14: renamed from D7; symbol open-automation:D_1N5819HW -> Open_Automation:D_1N5819HW; LCSC (none) -> C117948
- J11: renamed from J4; footprint open-automation:USB-mini-B-0548190519 -> Open_Automation:USB-mini-B-0548190519; symbol open-automation:USB_MINI_B -> Open_Automation:USB_MINI_B
- R84: renamed from R4; footprint Resistor_SMD:R_0603_1608Metric_Pad1.05x0.95mm_HandSolder -> Resistor_SMD:R_0603_1608Metric_Pad0.98x0.95mm_HandSolder; symbol open-automation:R_27 -> Open_Automation:R_27; LCSC (none) -> C22966; Part Number ERJ-3GEYJ2R2V -> 0603WAF2700T5E
- R85: renamed from R5; footprint Resistor_SMD:R_0603_1608Metric_Pad1.05x0.95mm_HandSolder -> Resistor_SMD:R_0603_1608Metric_Pad0.98x0.95mm_HandSolder; symbol open-automation:R_27 -> Open_Automation:R_27; LCSC (none) -> C22966; Part Number ERJ-3GEYJ2R2V -> 0603WAF2700T5E
- R86: renamed from R6; footprint Resistor_SMD:R_0603_1608Metric_Pad1.05x0.95mm_HandSolder -> Resistor_SMD:R_0603_1608Metric_Pad0.98x0.95mm_HandSolder; symbol open-automation:R_10K -> Open_Automation:R_10K; LCSC (none) -> C25804; Part Number RC0603JR-0710KL -> 0603WAF1002T5E
- R87: renamed from R7; footprint Resistor_SMD:R_0603_1608Metric_Pad1.05x0.95mm_HandSolder -> Resistor_SMD:R_0603_1608Metric_Pad0.98x0.95mm_HandSolder; symbol open-automation:R_10K -> Open_Automation:R_10K; LCSC (none) -> C25804; Part Number RC0603JR-0710KL -> 0603WAF1002T5E
- U16: renamed from U6; symbol open-automation:FT231XS -> Open_Automation:FT231XS; LCSC (none) -> C132160
Connections:
- net labels added: VBUS
- wire segments 44 -> 48

Commit message: finished layout and routing
Parts:
- Q17: symbol Open_Automation:Q_NPN -> open-dash-daughterboard-rescue:Q_NPN-Open_Automation
- Q18: symbol Open_Automation:Q_PNP -> open-dash-daughterboard-rescue:Q_PNP-Open_Automation
Changed lines of the file:
@@
 $EndComp
 $Comp
-L Open_Automation:Q_PNP Q18
+L open-dash-daughterboard-rescue:Q_PNP-Open_Automation Q18
 U 1 1 601A5292
 P 7150 4250
@@
 $EndComp
 $Comp
-L Open_Automation:Q_NPN Q17
+L open-dash-daughterboard-rescue:Q_NPN-Open_Automation Q17
 U 1 1 601A478F
 P 7150 3700
