File: daughter/circuits/usb.sch (KiCad schematic (older format))
At the start: 30 parts, among them J15 USB_MINI_B, J16 Conn_02x02_Counter_Clockwise, J18 USB_MINI_B, J42 Conn_02x02_Counter_Clockwise, Q1 Q_NPN_BEC, Q2 Q_PNP_BEC, Q5 Crystal_12Mhz, Q6 Q_SS8050, Q7 Q_SS8550, U10 CH340T(SSOP20W), U12 FT231XS

Commit message: Using npn-pnp high side switch for ext amp trigger.
Parts:
- removed C28, C30: C_47pF, Capacitor_SMD:C_0603_1608Metric_Pad1.08x0.95mm_HandSolder, symbol Open_Automation:C_47pF
- removed C29, C31: C_0.1uF, Capacitor_SMD:C_0603_1608Metric_Pad1.08x0.95mm_HandSolder, symbol open-dash-daughterboard-rescue:C_0.1uF-Open_Automation
- removed C32: C_4.7uF, Capacitor_SMD:C_0805_2012Metric_Pad1.18x1.45mm_HandSolder, symbol Open_Automation:C_4.7uF
- removed D14: D_1N5819HW, Diode_SMD:D_SOD-123, symbol Open_Automation:D_1N5819HW
- removed J15: USB_MINI_B, Open_Automation:USB-mini-B-0548190519, symbol open-dash-daughterboard-rescue:USB_MINI_B-Open_Automation
- removed J16, J42: Conn_02x02_Counter_Clockwise, Connector_PinHeader_2.54mm:PinHeader_2x02_P2.54mm_Vertical, symbol open-dash-daughterboard-rescue:Conn_02x02_Counter_Clockwise-Connector_Generic
- removed Q1: Q_NPN_BEC, Package_TO_SOT_SMD:SOT-23, symbol Open_Automation:Q_NPN_BEC
- removed Q2: Q_PNP_BEC, Package_TO_SOT_SMD:SOT-23, symbol Open_Automation:Q_PNP_BEC
- removed R43, R44: R_27, Resistor_SMD:R_0603_1608Metric_Pad0.98x0.95mm_HandSolder, symbol Open_Automation:R_27
- removed R45, R46: R_10K_0402, Resistor_SMD:R_0402_1005Metric_Pad0.72x0.64mm_HandSolder, symbol Open_Automation:R_10K_0402
- removed U12: FT231XS, Package_SO:SSOP-20_3.9x8.7mm_P0.635mm, symbol open-dash-daughterboard-rescue:FT231XS-Open_Automation
- renumbered C10 to C41, C7 to C42, C8 to C43, C9 to C44, J18 to J15, Q5 to Q1, Q6 to Q2, Q7 to Q39, R41 to R45, R42 to R85, U10 to U12
Connections:
- net RXD: no longer R45.2, U12.4 (RXD)
- new net TXD: R45.2, U12.4 (RXD)
