File: daughter/circuits/open-dash-daughterboard.kicad_pcb (KiCad board)
At the start: 4 copper layers, 120.4 x 100.2 mm, 213 parts, among them J1 Conn_01x01_Female, J10 Barrel_Jack_OD5.5_ID2.5, J11 Barrel_Jack_OD5.5_ID2.5, J12 AudioJack_3.5TRS, J13 AudioJack_3.5TRS, J14 Conn_01x05, J15 USB_MINI_B, J16 Conn_02x02_Counter_Clockwise, J17 Conn_01x08, J18 C1, J19 Conn_01x08, J2 Conn_01x01_Female, J20 Conn_01x20, J21 Conn_01x20, J22 Conn_IDE_40, J23 Conn_01x08, J24 C2, J25 Conn_01x08, J26 Conn_01x20, J27 Conn_IDE_40, J28 Conn_01x20, J29 Conn_01x08, J3 Conn_01x01_Female, J30 C3, J31 Conn_01x08, J32 Conn_IDE_40, J33 Conn_01x20, J34 Conn_01x20, J35 Conn_01x12, J36 STEREO, J37 Conn_01x12, J38 Conn_01x01_Female, J39 Conn_01x01_Female, J4 Conn_01x01_Female, J40 Conn_01x01_Female, J41 Conn_01x01_Female, J5 Conn_02x09_Odd_Even, J6 Conn_IDE_40, J7 Conn_IDE_40, J8 Conn_IDE_40, J9 Barrel_Jack_OD5.5_ID2.5, Q1 Q_NPN_BEC, Q10 Q_NPN_BEC, Q11 Q_DMHC4035LSD, Q12 Q_NPN_BEC, Q13 Q_NPN_BEC, Q14 Q_DMHC4035LSD, Q15 Q_NPN_BEC, Q16 Q_NPN_BEC, Q17 Q_DMHC4035LSD, Q18 Q_NPN_BEC, Q19 Q_NPN_BEC, Q2 Q_PNP_BEC, Q20 Q_DMHC4035LSD, Q21 Q_NPN_BEC, Q22 Q_NPN_BEC, Q23 Q_DMHC4035LSD, Q3 Q_NPN_BEC, Q4 Q_NPN_BEC, Q5 Q_NPN_BEC, Q6 Q_NPN_BEC, Q7 Q_NPN_BEC, Q8 Q_NPN_BEC, Q9 Q_NPN_BEC, SW1 SW_PUSH, SW2 SW_PUSH, SW3 SW_PUSH, T1 Audio_Transformer, T2 Audio_Transformer, T3 Audio_Transformer, T4 Audio_Transformer, U1 LTV-827S, U10 Si7020-A20, U11 MCP2551-I_SN, U12 FT231XS, U13 MCP23017_SS, U14 MAX11617, U2 ACS711, U3 REG_3V3, U4 MIC29302WU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

Commit message: finished schematic, working on layout
Parts:
- removed SW1, SW2, SW3: SW_PUSH, Button_Switch_SMD:SW_SPST_PTS645
- added C32: C_4.7uF, Capacitor_SMD:C_0805_2012Metric_Pad1.18x1.45mm_HandSolder, F.Cu at (205.8, 53.4)
- added C33: C_470uF, Capacitor_SMD:CP_Elec_10x10, F.Cu at (108.3, 115.1)
- added C34: C_470uF, Capacitor_SMD:CP_Elec_10x10, F.Cu at (104.1, 127.2)
- added EN1: SW_PUSH, Button_Switch_SMD:SW_SPST_PTS645, F.Cu at (128.5, 85.6)
- added FACT1: SW_PUSH, Button_Switch_SMD:SW_SPST_PTS645, F.Cu at (128.5, 67.7)
- added J42: Conn_02x02_Counter_Clockwise, Connector_PinHeader_2.54mm:PinHeader_2x02_P2.54mm_Vertical, F.Cu at (170.4, 71.7)
- added J43: Conn_02x02_Counter_Clockwise, Connector_PinHeader_2.54mm:PinHeader_2x02_P2.54mm_Vertical_SMD, F.Cu at (159.0, 101.6)
- added PROG1: SW_PUSH, Button_Switch_SMD:SW_SPST_PTS645, F.Cu at (128.3, 77.1)
- C1: value C_1000uF -> C_470uF; footprint Capacitor_THT:CP_Radial_D12.5mm_P5.00mm -> Capacitor_SMD:CP_Elec_10x10
- C10, C22: value C_1uF -> C_10uF; footprint Capacitor_SMD:C_0603_1608Metric_Pad1.08x0.95mm_HandSolder -> Capacitor_SMD:C_0805_2012Metric_Pad1.18x1.45mm_HandSolder
- C11, C13, C14, C15: footprint Capacitor_SMD:C_0603_1608Metric_Pad1.08x0.95mm_HandSolder -> Capacitor_SMD:C_0402_1005Metric_Pad0.74x0.62mm_HandSolder
- C12, C20, C23: value C_0.1uF -> C_1uF; footprint Capacitor_SMD:C_0603_1608Metric_Pad1.08x0.95mm_HandSolder -> Capacitor_SMD:C_0402_1005Metric_Pad0.74x0.62mm_HandSolder
- C16, C21: value C_10uF -> C_0.1uF; footprint Capacitor_SMD:C_0603_1608Metric_Pad1.08x0.95mm_HandSolder -> Capacitor_SMD:C_0402_1005Metric_Pad0.74x0.62mm_HandSolder
- C17: value C_470uF -> C_10uF; footprint Capacitor_THT:CP_Radial_D8.0mm_P3.50mm -> Capacitor_SMD:C_0805_2012Metric_Pad1.18x1.45mm_HandSolder
- C19: value C_1uF -> C_470uF; footprint Capacitor_SMD:C_0603_1608Metric_Pad1.08x0.95mm_HandSolder -> Capacitor_SMD:CP_Elec_10x10
- C2: value C_10uF -> C_470uF; footprint Capacitor_SMD:C_0603_1608Metric_Pad1.08x0.95mm_HandSolder -> Capacitor_SMD:CP_Elec_10x10
- C25: value C_560pF -> C_0.1uF; footprint Capacitor_SMD:C_0603_1608Metric_Pad1.08x0.95mm_HandSolder -> Capacitor_SMD:C_0402_1005Metric_Pad0.74x0.62mm_HandSolder
- C26: value C_560pF -> C_470pF
- C27: value C_47pF -> C_470pF
- C3, C4, C5, C6: footprint Capacitor_SMD:C_0603_1608Metric_Pad1.08x0.95mm_HandSolder -> Capacitor_SMD:C_0805_2012Metric_Pad1.18x1.45mm_HandSolder
- C30: value C_4.7uF -> C_47pF
- J18, J24, J30, J35, J36, J37: moved to B.Cu
- J5: value Conn_02x09_Odd_Even -> Conn_02x06_Odd_Even; footprint Connector_PinHeader_2.54mm:PinHeader_2x09_P2.54mm_Vertical_SMD -> Connector_PinHeader_2.54mm:PinHeader_2x06_P2.54mm_Vertical_SMD
- R10, R21, R32, R33, R34, R35, R36, R37, R39, R45, R46, R47, R48, R49, R50, R51, R52, R53, R54, R55: value R_10K -> R_10K_0402; footprint Resistor_SMD:R_0603_1608Metric_Pad0.98x0.95mm_HandSolder -> Resistor_SMD:R_0402_1005Metric_Pad0.72x0.64mm_HandSolder
- R22, R27: value R_47.5k -> R_47K_0402; footprint Resistor_SMD:R_0603_1608Metric_Pad0.98x0.95mm_HandSolder -> Resistor_SMD:R_0402_1005Metric_Pad0.72x0.64mm_HandSolder
- R38, R40: value R_4K7 -> R_4.7K; footprint Resistor_SMD:R_0603_1608Metric_Pad0.98x0.95mm_HandSolder -> Resistor_SMD:R_0402_1005Metric_Pad0.72x0.64mm_HandSolder
- R41, R42: footprint Resistor_SMD:R_0603_1608Metric_Pad0.98x0.95mm_HandSolder -> Resistor_SMD:R_0402_1005Metric_Pad0.72x0.64mm_HandSolder
- moved J15 271.5 mm to (196.7, 46.2), turned to 270 degrees
- moved J16 271.3 mm to (191.7, 52.0), turned to 90 degrees
- moved R44 269.7 mm to (203.1, 58.0), turned to 180 degrees
- moved D14 269.4 mm to (201.0, 53.5), turned to 180 degrees
- moved C29 262.9 mm to (206.6, 58.0)
- moved U12 259.7 mm to (202.9, 63.3), turned to 90 degrees
- moved R45 258.1 mm to (196.2, 60.7), turned to 270 degrees
- moved C30 257.0 mm to (203.1, 56.3)
- moved R43 255.8 mm to (199.5, 58.0), turned to 180 degrees
- moved C31 254.7 mm to (206.6, 56.3)
- moved J38 251.4 mm to (209.2, 202.9)
- moved R46 250.0 mm to (196.1, 65.3), turned to 90 degrees
- moved C28 249.3 mm to (199.5, 56.3)
- moved C27 245.8 mm to (185.6, 73.5), turned to 180 degrees
- moved Q1 245.5 mm to (193.6, 60.8), turned to 180 degrees
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Connections:
- C10 pad 1: /Audio Amplifier/MUTE -> /BATTERY
- C11 pad 1: /Audio Amplifier/STBY -> GND
- C11 pad 2: GND -> /Audio Amplifier/MUTE
- C12 pad 1: Net-(C12-Pad1) -> GND
- C12 pad 2: Net-(C12-Pad2) -> /Audio Amplifier/STBY
- C16 pad 1: /Audio Amplifier/SVR -> Net-(C16-Pad1)
- C16 pad 2: GND -> Net-(C16-Pad2)
- C17 pad 1: /BATTERY -> /Audio Amplifier/SVR
- C2 pad 1: /5V -> /BATTERY
- C20 pad 1: /BATTERY -> GND
- C20 pad 2: GND -> /BATTERY
- C21 pad 1: /3V3 -> /BATTERY
- C25 pad 1: Net-(C25-Pad1) -> /3V3
- C27 pad 1: /USB/USBDM -> Net-(C27-Pad1)
- C28 pad 1: /USB/USBDP -> /USB/USBDM
- C3 pad 1: /3V3 -> /5V
- C30 pad 1: /5V -> /USB/USBDP
- C4 pad 1: /BATTERY -> /3V3
- C5 pad 1: /Power/MAIN_POWER_IN -> /BATTERY
- C6 pad 1: /BATTERY -> /Power/MAIN_POWER_IN
- J20 pad 1: /Interface/J1850 -> /Interface/LEFT_AIR_TEMP_CONTROL_A
- J20 pad 10: /Interface/REAR_DEFOG -> /Interface/BATTERY
- J20 pad 11: /Interface/INSIDE_AIR_TEMP_BLOWER -> /Interface/LOWER_RIGHT_AIR_TEMP
- J20 pad 12: GND -> /Interface/WHEEL_CONTROLS_SIGNAL
- J20 pad 13: /Interface/LOW_REF -> /Interface/J1850
- J20 pad 14: /Interface/BATTERY -> /Interface/CAN+
- J20 pad 15: /Interface/BATTERY -> /Interface/CAN-
- J20 pad 16: /Interface/BATTERY -> /Interface/DISPLAY_POWER
- J20 pad 17: GND -> /Interface/MAIN_POWER
- J20 pad 2: /Interface/INSIDE_AIR_TEMP -> /Interface/LEFT_AIR_TEMP_CONTROL_B
- J20 pad 3: /Interface/UPPER_RIGHT_AIR_TEMP -> /Interface/RIGHT_AIR_TEMP_CONTROL_A
- J20 pad 4: /Interface/LOW_REF -> /Interface/RIGHT_AIR_TEMP_CONTROL_B
- J20 pad 5: /Interface/AMBIENT_AIR_TEMP -> /Interface/MODE_A
- J20 pad 6: /Interface/DRIVER_SUNLOAD -> /Interface/MODE_B
- J20 pad 7: /Interface/PASSENGER_SUNLOAD -> /Interface/RECIRCULATION_A
- J20 pad 8: /Interface/AMBIENT_LIGHT -> /Interface/RECIRCULATION_B
- J20 pad 9: /Interface/UPPER_LEFT_AIR_TEMP -> /Interface/BATTERY
- J21 pad 1: /Interface/PASSENGER_HEATED_SEAT_STATUS -> /Interface/LEFT_AIR_TEMP_CONTROL_A
- J21 pad 10: /Interface/TRIGGER1 -> /Interface/BATTERY
- J21 pad 11: /Interface/SENSE1 -> /Interface/LOWER_LEFT_AIR_TEMP
- J21 pad 12: GND -> /Interface/WHEEL_CONTROLS_SUPPLY
- J21 pad 13: /Interface/LOW_REF -> /Interface/IGNITION
- J21 pad 15: /Interface/BATTERY -> GND
- J21 pad 16: /Interface/BATTERY -> /Interface/DISPLAY_POWER
- J21 pad 17: GND -> /Interface/MAIN_POWER
- J21 pad 2: /Interface/DRIVER_HEATED_SEAT_STATUS -> /Interface/LEFT_AIR_TEMP_CONTROL_B
- J21 pad 3: /Interface/IGNITION -> /Interface/RIGHT_AIR_TEMP_CONTROL_A
- J21 pad 4: /Interface/BATTERY -> /Interface/RIGHT_AIR_TEMP_CONTROL_B
- J21 pad 5: /Interface/BLOWER_MOTOR -> /Interface/MODE_A
- J21 pad 6: /Interface/PASSENGER_SEAT_TEMP_CONTROL -> /Interface/MODE_B
- J21 pad 7: /Interface/DRIVER_SEAT_TEMP_CONTROL -> /Interface/RECIRCULATION_A
- J21 pad 8: /Interface/INSTRUMENT_SUPPLY_VOLTAGE_4 -> /Interface/RECIRCULATION_B
- J22 pad 1: /Interface/J1850 -> /Interface/LEFT_AIR_TEMP_CONTROL_A
- J22 pad 10: /Interface/BLOWER_MOTOR -> /Interface/MODE_A
- J22 pad 11: /Interface/DRIVER_SUNLOAD -> /Interface/MODE_B
- J22 pad 12: /Interface/PASSENGER_SEAT_TEMP_CONTROL -> /Interface/MODE_B
- J22 pad 13: /Interface/PASSENGER_SUNLOAD -> /Interface/RECIRCULATION_A
- J22 pad 14: /Interface/DRIVER_SEAT_TEMP_CONTROL -> /Interface/RECIRCULATION_A
- J22 pad 15: /Interface/AMBIENT_LIGHT -> /Interface/RECIRCULATION_B
- J22 pad 16: /Interface/INSTRUMENT_SUPPLY_VOLTAGE_4 -> /Interface/RECIRCULATION_B
- J22 pad 17: /Interface/UPPER_LEFT_AIR_TEMP -> /Interface/BATTERY
- J22 pad 19: /Interface/REAR_DEFOG -> /Interface/BATTERY
- J22 pad 2: /Interface/PASSENGER_HEATED_SEAT_STATUS -> /Interface/LEFT_AIR_TEMP_CONTROL_A
- J22 pad 20: /Interface/TRIGGER1 -> /Interface/BATTERY
- J22 pad 21: /Interface/INSIDE_AIR_TEMP_BLOWER -> /Interface/LOWER_RIGHT_AIR_TEMP
- J22 pad 22: /Interface/SENSE1 -> /Interface/LOWER_LEFT_AIR_TEMP
- J22 pad 23: GND -> /Interface/WHEEL_CONTROLS_SIGNAL
- J22 pad 24: GND -> /Interface/WHEEL_CONTROLS_SUPPLY
- J22 pad 25: /Interface/LOW_REF -> /Interface/J1850
- J22 pad 26: /Interface/LOW_REF -> /Interface/IGNITION
- J22 pad 27: /Interface/BATTERY -> /Interface/CAN+
- J22 pad 29: /Interface/BATTERY -> /Interface/CAN-
- J22 pad 3: /Interface/INSIDE_AIR_TEMP -> /Interface/LEFT_AIR_TEMP_CONTROL_B
- J22 pad 30: /Interface/BATTERY -> GND
- J22 pad 31: /Interface/BATTERY -> /Interface/DISPLAY_POWER
- J22 pad 32: /Interface/BATTERY -> /Interface/DISPLAY_POWER
- J22 pad 33: GND -> /Interface/MAIN_POWER
- J22 pad 34: GND -> /Interface/MAIN_POWER
- J22 pad 4: /Interface/DRIVER_HEATED_SEAT_STATUS -> /Interface/LEFT_AIR_TEMP_CONTROL_B
- J22 pad 5: /Interface/UPPER_RIGHT_AIR_TEMP -> /Interface/RIGHT_AIR_TEMP_CONTROL_A
- J22 pad 6: /Interface/IGNITION -> /Interface/RIGHT_AIR_TEMP_CONTROL_A
- J22 pad 7: /Interface/LOW_REF -> /Interface/RIGHT_AIR_TEMP_CONTROL_B
- J22 pad 8: /Interface/BATTERY -> /Interface/RIGHT_AIR_TEMP_CONTROL_B
- J22 pad 9: /Interface/AMBIENT_AIR_TEMP -> /Interface/MODE_A
- J26 pad 1: /Interface/LEFT_AIR_TEMP_CONTROL_A -> /Interface/BATTERY
- J26 pad 10: /Interface/BATTERY -> /Interface/LR-
- J26 pad 11: GND -> /Interface/RR+
- J26 pad 12: /Interface/WHEEL_CONTROLS_SIGNAL -> /Interface/RR-
- J26 pad 13: /Interface/DISPLAY_POWER -> /Interface/AUDIO_IN4
- J26 pad 14: /Interface/MAIN_POWER -> /Interface/AUDIO_IN3
- J26 pad 15: /Interface/CAN+ -> /Interface/AUDIO_IN2
- J26 pad 16: /Interface/IGNITION -> /Interface/AUDIO_IN1
- J26 pad 17: /Interface/BATTERY -> GND
- J26 pad 18: /Interface/BATTERY -> GND
- J26 pad 2: /Interface/LEFT_AIR_TEMP_CONTROL_A -> /Interface/BATTERY
- J26 pad 3: /Interface/RIGHT_AIR_TEMP_CONTROL_A -> /Interface/BATTERY
- J26 pad 4: /Interface/RIGHT_AIR_TEMP_CONTROL_A -> /Interface/BATTERY
- J26 pad 5: /Interface/MODE_A -> /Interface/LF+
- J26 pad 6: /Interface/MODE_A -> /Interface/LF-
- J26 pad 7: /Interface/RECIRCULATION_A -> /Interface/RF+
- J26 pad 8: /Interface/RECIRCULATION_A -> /Interface/RF-
- J26 pad 9: /Interface/LOWER_LEFT_AIR_TEMP -> /Interface/LR+
- J27 pad 1: /Interface/LEFT_AIR_TEMP_CONTROL_A -> /Interface/BATTERY
- J27 pad 10: /Interface/MODE_B -> /Interface/LF+
- J27 pad 11: /Interface/MODE_A -> /Interface/LF-
- J27 pad 12: /Interface/MODE_B -> /Interface/LF-
- J27 pad 13: /Interface/RECIRCULATION_A -> /Interface/RF+
- J27 pad 14: /Interface/RECIRCULATION_B -> /Interface/RF+
- J27 pad 15: /Interface/RECIRCULATION_A -> /Interface/RF-
- J27 pad 16: /Interface/RECIRCULATION_B -> /Interface/RF-
- J27 pad 17: /Interface/LOWER_LEFT_AIR_TEMP -> /Interface/LR+
- J27 pad 18: /Interface/LOWER_RIGHT_AIR_TEMP -> /Interface/LR+
- J27 pad 19: /Interface/BATTERY -> /Interface/LR-
- J27 pad 2: /Interface/LEFT_AIR_TEMP_CONTROL_B -> /Interface/BATTERY
- J27 pad 20: /Interface/BATTERY -> /Interface/LR-
- J27 pad 21: GND -> /Interface/RR+
- J27 pad 22: GND -> /Interface/RR+
- J27 pad 23: /Interface/WHEEL_CONTROLS_SIGNAL -> /Interface/RR-
- J27 pad 24: /Interface/WHEEL_CONTROLS_SUPPLY -> /Interface/RR-
- J27 pad 25: /Interface/DISPLAY_POWER -> /Interface/AUDIO_IN4
- J27 pad 26: /Interface/DISPLAY_POWER -> /Interface/AUDIO_IN4
- J27 pad 27: /Interface/MAIN_POWER -> /Interface/AUDIO_IN3
- J27 pad 28: /Interface/MAIN_POWER -> /Interface/AUDIO_IN3
- J27 pad 29: /Interface/CAN+ -> /Interface/AUDIO_IN2
- J27 pad 3: /Interface/LEFT_AIR_TEMP_CONTROL_A -> /Interface/BATTERY
- J27 pad 30: /Interface/CAN- -> /Interface/AUDIO_IN2
- J27 pad 31: /Interface/IGNITION -> /Interface/AUDIO_IN1
- J27 pad 32: /Interface/J1850 -> /Interface/AUDIO_IN1
- J27 pad 33: /Interface/BATTERY -> GND
- J27 pad 34: /Interface/BATTERY -> GND
- J27 pad 35: /Interface/BATTERY -> GND
- J27 pad 36: /Interface/BATTERY -> GND
- J27 pad 4: /Interface/LEFT_AIR_TEMP_CONTROL_B -> /Interface/BATTERY
- J27 pad 5: /Interface/RIGHT_AIR_TEMP_CONTROL_A -> /Interface/BATTERY
- J27 pad 6: /Interface/RIGHT_AIR_TEMP_CONTROL_B -> /Interface/BATTERY
- J27 pad 7: /Interface/RIGHT_AIR_TEMP_CONTROL_A -> /Interface/BATTERY
- J27 pad 8: /Interface/RIGHT_AIR_TEMP_CONTROL_B -> /Interface/BATTERY
- J27 pad 9: /Interface/MODE_A -> /Interface/LF+
- J28 pad 1: /Interface/LEFT_AIR_TEMP_CONTROL_B -> /Interface/BATTERY
- J28 pad 10: /Interface/BATTERY -> /Interface/LR-
- J28 pad 11: GND -> /Interface/RR+
- J28 pad 12: /Interface/WHEEL_CONTROLS_SUPPLY -> /Interface/RR-
- J28 pad 13: /Interface/DISPLAY_POWER -> /Interface/AUDIO_IN4
- J28 pad 14: /Interface/MAIN_POWER -> /Interface/AUDIO_IN3
- J28 pad 15: /Interface/CAN- -> /Interface/AUDIO_IN2
- J28 pad 16: /Interface/J1850 -> /Interface/AUDIO_IN1
- J28 pad 17: /Interface/BATTERY -> GND
- J28 pad 18: /Interface/BATTERY -> GND
- J28 pad 2: /Interface/LEFT_AIR_TEMP_CONTROL_B -> /Interface/BATTERY
- J28 pad 3: /Interface/RIGHT_AIR_TEMP_CONTROL_B -> /Interface/BATTERY
- J28 pad 4: /Interface/RIGHT_AIR_TEMP_CONTROL_B -> /Interface/BATTERY
- J28 pad 5: /Interface/MODE_B -> /Interface/LF+
- J28 pad 6: /Interface/MODE_B -> /Interface/LF-
- J28 pad 7: /Interface/RECIRCULATION_B -> /Interface/RF+
- J28 pad 8: /Interface/RECIRCULATION_B -> /Interface/RF-
- J28 pad 9: /Interface/LOWER_RIGHT_AIR_TEMP -> /Interface/LR+
- J32 pad 1: /Interface/BATTERY -> /Interface/J1850
- J32 pad 10: /Interface/LR+ -> /Interface/BLOWER_MOTOR
- J32 pad 11: /Interface/LF- -> /Interface/DRIVER_SUNLOAD
- J32 pad 12: /Interface/LR- -> /Interface/PASSENGER_SEAT_TEMP_CONTROL
- J32 pad 13: /Interface/LF- -> /Interface/PASSENGER_SUNLOAD
- J32 pad 14: /Interface/LR- -> /Interface/DRIVER_SEAT_TEMP_CONTROL
- J32 pad 15: /Interface/LF- -> /Interface/AMBIENT_LIGHT
- J32 pad 16: /Interface/LR- -> /Interface/INSTRUMENT_SUPPLY_VOLTAGE_4
- J32 pad 17: /Interface/RR- -> /Interface/UPPER_LEFT_AIR_TEMP
- J32 pad 18: /Interface/RF- -> /Interface/BATTERY
- J32 pad 19: /Interface/RR- -> /Interface/REAR_DEFOG
- J32 pad 2: /Interface/BATTERY -> /Interface/PASSENGER_HEATED_SEAT_STATUS
- J32 pad 20: /Interface/RF- -> /Interface/TRIGGER1
- J32 pad 21: /Interface/RR- -> /Interface/INSIDE_AIR_TEMP_BLOWER
- J32 pad 22: /Interface/RF- -> /Interface/SENSE1
- J32 pad 23: /Interface/RR+ -> GND
- J32 pad 24: /Interface/RF+ -> GND
- J32 pad 25: /Interface/RR+ -> /Interface/LOW_REF
- J32 pad 26: /Interface/RF+ -> /Interface/LOW_REF
- J32 pad 27: /Interface/RR+ -> /Interface/BATTERY
- J32 pad 28: /Interface/RF+ -> /Interface/BATTERY
- J32 pad 29: /Interface/AUDIO_IN1 -> /Interface/BATTERY
- J32 pad 3: /Interface/BATTERY -> /Interface/INSIDE_AIR_TEMP
- J32 pad 30: /Interface/AUDIO_IN3 -> /Interface/BATTERY
- J32 pad 31: /Interface/AUDIO_IN1 -> /Interface/BATTERY
- J32 pad 32: /Interface/AUDIO_IN3 -> /Interface/BATTERY
- J32 pad 33: /Interface/AUDIO_IN2 -> GND
- J32 pad 34: /Interface/AUDIO_IN4 -> GND
- J32 pad 35: /Interface/AUDIO_IN2 -> GND
- J32 pad 36: /Interface/AUDIO_IN4 -> GND
- J32 pad 4: /Interface/BATTERY -> /Interface/DRIVER_HEATED_SEAT_STATUS
- J32 pad 5: /Interface/LF+ -> /Interface/UPPER_RIGHT_AIR_TEMP
- J32 pad 6: /Interface/LR+ -> /Interface/IGNITION
- J32 pad 7: /Interface/LF+ -> /Interface/LOW_REF
- J32 pad 8: /Interface/LR+ -> /Interface/BATTERY
- J32 pad 9: /Interface/LF+ -> /Interface/AMBIENT_AIR_TEMP
- J33 pad 1: /Interface/BATTERY -> /Interface/J1850
- J33 pad 10: /Interface/RR- -> /Interface/REAR_DEFOG
- J33 pad 11: /Interface/RR- -> /Interface/INSIDE_AIR_TEMP_BLOWER
- J33 pad 12: /Interface/RR+ -> GND
- J33 pad 13: /Interface/RR+ -> /Interface/LOW_REF
- J33 pad 14: /Interface/RR+ -> /Interface/BATTERY
- J33 pad 15: /Interface/AUDIO_IN1 -> /Interface/BATTERY
- J33 pad 16: /Interface/AUDIO_IN1 -> /Interface/BATTERY
- J33 pad 17: /Interface/AUDIO_IN2 -> GND
- J33 pad 18: /Interface/AUDIO_IN2 -> GND
- J33 pad 2: /Interface/BATTERY -> /Interface/INSIDE_AIR_TEMP
- J33 pad 3: /Interface/LF+ -> /Interface/UPPER_RIGHT_AIR_TEMP
- J33 pad 4: /Interface/LF+ -> /Interface/LOW_REF
- J33 pad 5: /Interface/LF+ -> /Interface/AMBIENT_AIR_TEMP
- J33 pad 6: /Interface/LF- -> /Interface/DRIVER_SUNLOAD
- J33 pad 7: /Interface/LF- -> /Interface/PASSENGER_SUNLOAD
- J33 pad 8: /Interface/LF- -> /Interface/AMBIENT_LIGHT
- J33 pad 9: /Interface/RR- -> /Interface/UPPER_LEFT_AIR_TEMP
- J34 pad 1: /Interface/BATTERY -> /Interface/PASSENGER_HEATED_SEAT_STATUS
- J34 pad 10: /Interface/RF- -> /Interface/TRIGGER1
- J34 pad 11: /Interface/RF- -> /Interface/SENSE1
- J34 pad 12: /Interface/RF+ -> GND
- J34 pad 13: /Interface/RF+ -> /Interface/LOW_REF
- J34 pad 14: /Interface/RF+ -> /Interface/BATTERY
- J34 pad 15: /Interface/AUDIO_IN3 -> /Interface/BATTERY
- J34 pad 16: /Interface/AUDIO_IN3 -> /Interface/BATTERY
- J34 pad 17: /Interface/AUDIO_IN4 -> GND
- J34 pad 18: /Interface/AUDIO_IN4 -> GND
- J34 pad 2: /Interface/BATTERY -> /Interface/DRIVER_HEATED_SEAT_STATUS
- J34 pad 3: /Interface/LR+ -> /Interface/IGNITION
- J34 pad 4: /Interface/LR+ -> /Interface/BATTERY
- J34 pad 5: /Interface/LR+ -> /Interface/BLOWER_MOTOR
- J34 pad 6: /Interface/LR- -> /Interface/PASSENGER_SEAT_TEMP_CONTROL
- J34 pad 7: /Interface/LR- -> /Interface/DRIVER_SEAT_TEMP_CONTROL
- J34 pad 8: /Interface/LR- -> /Interface/INSTRUMENT_SUPPLY_VOLTAGE_4
- J34 pad 9: /Interface/RF- -> /Interface/BATTERY
- J5 pad 1: GND -> /BATTERY
- J5 pad 10: /TXD -> /AIN9
- J5 pad 11: /5V -> GND
- J5 pad 12: /RXD -> GND
- J5 pad 2: /OUT11 -> /BATTERY
- J5 pad 4: /AIN10 -> /5V
- J5 pad 5: /FACT -> /3V3
- J5 pad 6: /SDA -> /3V3
- J5 pad 7: /ESP_EN -> /FACT
- J5 pad 8: /SCL -> /AIN10
- J5 pad 9: /3V3 -> /C_OUT3
- J6 pad 10: /MODE_B -> /MODE_A
- J6 pad 11: /MODE_A -> /MODE_B
- J6 pad 14: /RECIRCULATION_B -> /RECIRCULATION_A
- J6 pad 15: /RECIRCULATION_A -> /RECIRCULATION_B
- J6 pad 17: /LOWER_LEFT_AIR_TEMP -> /BATTERY
- J6 pad 18: /LOWER_RIGHT_AIR_TEMP -> /BATTERY
- J6 pad 2: /LEFT_AIR_TEMP_CONTROL_B -> /LEFT_AIR_TEMP_CONTROL_A
- J6 pad 21: GND -> /LOWER_RIGHT_AIR_TEMP
- J6 pad 22: GND -> /LOWER_LEFT_AIR_TEMP
- J6 pad 25: /DISPLAY_POWER -> /J1850
- J6 pad 26: /DISPLAY_POWER -> /IGNITION
- J6 pad 27: /MAIN_POWER -> /CAN+
- J6 pad 28: /MAIN_POWER -> /BATTERY
- J6 pad 29: /CAN+ -> /CAN-
- J6 pad 3: /LEFT_AIR_TEMP_CONTROL_A -> /LEFT_AIR_TEMP_CONTROL_B
- J6 pad 30: /CAN- -> GND
- J6 pad 31: /IGNITION -> /DISPLAY_POWER
- J6 pad 32: /J1850 -> /DISPLAY_POWER
- J6 pad 33: /BATTERY -> /MAIN_POWER
- J6 pad 34: /BATTERY -> /MAIN_POWER
- J6 pad 35: /BATTERY -> GND
- J6 pad 36: /BATTERY -> GND
- J6 pad 6: /RIGHT_AIR_TEMP_CONTROL_B -> /RIGHT_AIR_TEMP_CONTROL_A
- J6 pad 7: /RIGHT_AIR_TEMP_CONTROL_A -> /RIGHT_AIR_TEMP_CONTROL_B
- J7 pad 10: /LR+ -> /LF+
- J7 pad 12: /LR- -> /LF-
- J7 pad 13: /LF- -> /RF+
- J7 pad 14: /LR- -> /RF+
- J7 pad 15: /LF- -> /RF-
- J7 pad 16: /LR- -> /RF-
- J7 pad 17: /RR- -> /LR+
- J7 pad 18: /RF- -> /LR+
- J7 pad 19: /RR- -> /LR-
- J7 pad 20: /RF- -> /LR-
- J7 pad 21: /RR- -> /RR+
- J7 pad 22: /RF- -> /RR+
- J7 pad 23: /RR+ -> /RR-
- J7 pad 24: /RF+ -> /RR-
- J7 pad 25: /RR+ -> /AUDIO_IN4
- J7 pad 26: /RF+ -> /AUDIO_IN4
- J7 pad 27: /RR+ -> /AUDIO_IN3
- J7 pad 28: /RF+ -> /AUDIO_IN3
- J7 pad 29: /AUDIO_IN1 -> /AUDIO_IN2
- J7 pad 30: /AUDIO_IN3 -> /AUDIO_IN2
- J7 pad 32: /AUDIO_IN3 -> /AUDIO_IN1
- J7 pad 33: /AUDIO_IN2 -> GND
- J7 pad 34: /AUDIO_IN4 -> GND
- J7 pad 35: /AUDIO_IN2 -> GND
- J7 pad 36: /AUDIO_IN4 -> GND
- J7 pad 5: /LF+ -> /BATTERY
- J7 pad 6: /LR+ -> /BATTERY
- J7 pad 7: /LF+ -> /BATTERY
- J7 pad 8: /LR+ -> /BATTERY
- Q5 pad 3: /INSIDE_AIR_TEMP_BLOWER -> /REAR_DEFOG
- Q7 pad 3: /INSIDE_AIR_TEMP_BLOWER -> /C_OUT3
- R10 pad 1: /3V3 -> /DISPLAY_EN
- R10 pad 2: /DISPLAY_EN -> /3V3
- R21 pad 1: /Audio Amplifier/STBY -> /AUDIO_STBY
- R21 pad 2: /AUDIO_STBY -> /Audio Amplifier/STBY
- R22 pad 1: /AUDIO_MUTE -> /Audio Amplifier/MUTE
- R22 pad 2: /Audio Amplifier/MUTE -> /AUDIO_MUTE
- R23 pad 1: Net-(C12-Pad1) -> Net-(C13-Pad2)
- R24 pad 1: Net-(C13-Pad1) -> Net-(C14-Pad2)
- R25 pad 1: Net-(C14-Pad1) -> Net-(C15-Pad2)
- R26 pad 1: Net-(C15-Pad1) -> Net-(C16-Pad2)
- R27 pad 1: /Audio Amplifier/OD -> GND
- R27 pad 2: GND -> /Audio Amplifier/OD
- R35 pad 1: GND -> /Microcontroller/IO2
- R35 pad 2: /Microcontroller/IO2 -> GND
- R37 pad 1: /3V3 -> /SCL
- R37 pad 2: /SCL -> /3V3
- R38 pad 1: /CANbus/RX -> /CAN_RX
- R38 pad 2: /CAN_RX -> /CANbus/RX
- R40 pad 1: Net-(R40-Pad1) -> GND
- R40 pad 2: GND -> Net-(R40-Pad2)
- R41 pad 1: Net-(C25-Pad1) -> Net-(C26-Pad1)
- R42 pad 1: Net-(C26-Pad1) -> Net-(C27-Pad1)
- R45 pad 1: Net-(Q2-Pad1) -> Net-(Q1-Pad1)
- R45 pad 2: /USB/RTS -> /USB/DTR
- R46 pad 1: /USB/DTR -> Net-(Q2-Pad1)
- R46 pad 2: Net-(Q1-Pad1) -> /USB/RTS
- U11 pad 8: Net-(R40-Pad1) -> Net-(R40-Pad2)
- U13 pad 19: /IO26 -> /INTB
- U13 pad 20: /IO25 -> /INTA
- U7 pad 11: Net-(C12-Pad2) -> Net-(C13-Pad1)
- U7 pad 12: Net-(C13-Pad2) -> Net-(C14-Pad1)
- U7 pad 14: Net-(C15-Pad2) -> Net-(C16-Pad1)
- U7 pad 15: Net-(C14-Pad2) -> Net-(C15-Pad1)
- U9 pad 10: /IO25 -> /INTA
- U9 pad 11: /IO26 -> /INTB
Other:
- board size 120.4 x 100.2 mm -> 125.1 x 162.3 mm
